Commit message: Draw the 6 cm safety cushion as a visual-only URDF link
Makes the stop condition visible instead of inferred: a translucent
0.48 x 1.12 m rectangle at floor level, which is the chassis plus 6 cm all
round. When a /scan_reliable return crosses inside it, the robot is at the
cushion boundary in that direction -- the exact condition the guarded-drive
feature will act on.

Verified equal to nav2_params.yaml's costmap footprint polygon on both
costmaps, and the margin checked as exactly 6.0 cm per side on both axes.
Flagged inline as a mirror rather than a source: the numbers are duplicated
from the Nav2 config and nothing enforces they stay in step, so once Nav2
runs, local_costmap/published_footprint is the authoritative version --
correct by construction, since the planner publishes what it actually
collision-checks. This link is what gives the picture beforehand, and
remains useful afterwards during teleop when Nav2 is not running.

Visual only, with no collision element so Gazebo cannot mistake a safety
margin for a physical object, and no inertial, following base_footprint's
precedent for massless fixed-joint links.

Context: driving the robot to a wall and measuring gave ~7 cm by tape
against 0.06-0.07 m read off Foxglove. That agreement validates the whole
geometry chain end-to-end -- range, the mirror+270 angular correction, the
0.27 m laser offset, the 0.36 m chassis width, and base_link's placement --
and is the first check to confirm scale and offset rather than only
direction, which is all the earlier orientation work could establish.

Co-Authored-By: Claude Sonnet 5 <noreply@anthropic.com>
Claude-Session: https://claude.ai/code/session_01GXZfYqdSmqvc5WQ8g2cGg9

File: src/mecanum_robot/urdf/aislebot.urdf (robot description, URDF)
Before this commit: robot aislebot, 9 links, 8 joints
Links:
- added link safety_cushion; visual box size=0.48 1.12 0.01
Joints:
- added joint safety_cushion_joint: type fixed, parent base_link, child safety_cushion, origin xyz=0 0 0.005 rpy=0 0 0

Commit message: Sync the Pi's newer files into the repo (state of 17 Oct 2026)
These nine files were changed on the Pi after their last repo commit
(Pi modification times 6 Oct 2026, the axis refactor to REP-103 and the
dashboard work) and never came back. Copied read-only over the ro key; each
file's sha256 on the Pi equals the local copy byte for byte.

  src/mecanum_navigation/config/nav2_params.yaml
  src/mecanum_navigation/launch/nav2_slam.launch.py
  src/mecanum_navigation/launch/navigation.launch.py
  src/mecanum_robot/launch/sensors.launch.py
  src/mecanum_robot/mecanum_robot/odometry_publisher.py
  src/mecanum_robot/mecanum_robot/phone_dashboard.py
  src/mecanum_robot/urdf/aislebot.urdf
  src/scan_relay/scan_relay.py
  tools/nav_goal.py

tools/tests/dashboard_html_syntax.py passes on the dashboard (node --check on
the runtime string, no stray backslashes). That is not a browser check.

Not done: the docs these files refer to (e.g. docs/Axis_Refactor_Plan.md) are
not in the repo, and about seven tools on the Pi's ros2_ws/tools are not in
the repo either.

Co-Authored-By: Claude Sonnet 5.5 <noreply@anthropic.com>

File: src/mecanum_robot/urdf/aislebot.urdf (robot description, URDF)
Before this commit: robot aislebot, 10 links, 9 joints
Links:
- link chassis: geometry collision box size=1.0 0.36 0.15; visual box size=1.0 0.36 0.15
- link safety_cushion: geometry visual box size=1.12 0.48 0.01
Joints:
- joint laser_joint: origin xyz=0 0.27 0.275 rpy=0 0 0 -> xyz=0.27 0 0.275 rpy=0 0 0
- joint wheel_fl_joint: axis 1 0 0 -> 0 1 0; origin xyz=-0.15769 0.333 0 rpy=0 0 0 -> xyz=0.333 0.15769 0 rpy=0 0 0
- joint wheel_fr_joint: axis 1 0 0 -> 0 1 0; origin xyz=0.15769 0.403 0 rpy=0 0 0 -> xyz=0.403 -0.15769 0 rpy=0 0 0
- joint wheel_rl_joint: axis 1 0 0 -> 0 1 0; origin xyz=-0.15769 -0.403 0 rpy=0 0 0 -> xyz=-0.403 0.15769 0 rpy=0 0 0
- joint wheel_rr_joint: axis 1 0 0 -> 0 1 0; origin xyz=0.15769 -0.333 0 rpy=0 0 0 -> xyz=-0.333 -0.15769 0 rpy=0 0 0
